File: tests/NexRx/NexRx_routed.kicad_pcb (KiCad board)
At the start: 3 copper layers, 349 parts

Commit message: Increase SimpleGridRouter iteration limit as temporary perf fix
TEMPORARY FIX for slow routing performance. This is NOT a proper solution.

Changes:
- Increased max iterations from 10,000 to 100,000 (10x)
- Added early termination when within 2 grid cells of goal
- Added TODO comments marking this as temporary

ROOT CAUSE:
MazeSearchAlgo.cpp (line 87-138) is using SimpleGridRouter as a fallback
instead of implementing the proper expansion room algorithm from Java.

SimpleGridRouter is fundamentally slower:
- Grid-based A*: explores O(W×H×L) cells = millions for complex boards
- Java expansion rooms: explore O(R×D) = hundreds of rooms/doors
- Linear parent lookups: O(N) per expansion
- No door-based pruning, drill page indexing, or room completion

This 10x increase helps simple boards but complex boards like NexRx (1148 items)
will still take hours instead of minutes.

REAL FIX NEEDED:
Must port expansion room infrastructure from Java:
1. Room generation (CompleteExpansionRoom, FreeSpaceExpansionRoom)
2. Door calculation (SortedOrthogonalRoomNeighbours)
3. Drill page arrays for via optimization
4. Proper maze expansion loop with priority queue and pruning

See: freerouting.app/src/main/java/app/freerouting/autoroute/MazeSearchAlgo.java
     (1290 lines vs our 308-line stub)

🤖 Generated with [Claude Code](https://claude.com/claude-code)

Co-Authored-By: Claude <noreply@anthropic.com>
Routing:
- net +3.3V: track 17100.0 -> 2633.4 mm, vias 0 -> 719
- net +2V5bias: track 4200.0 -> 833.4 mm, vias 0 -> 321
- net /Rx Front End/Rx Preselector/preselIn: track 3700.0 -> 945.4 mm, vias 0 -> 208
- net +1V65bias: track 2320.0 -> 417.6 mm, vias 0 -> 142
- net +3.3VFPGAIO: track 2200.0 -> 561.5 mm, vias 0 -> 193
- net /FPGA/Ctrl.qsdMOSI: track 1600.0 -> 137.6 mm, vias 0 -> 69
- net /FPGA/Ctrl.qsdSCK: track 1600.0 -> 163.6 mm, vias 0 -> 59
- net +3.3V-ON: track 2000.0 -> 627.9 mm, vias 0 -> 280
- net /FPGA/Ctrl.qsdNSS: track 1500.0 -> 242.3 mm, vias 0 -> 92
- net /FPGA/FPGA.NSS: track 1000.0 -> 162.9 mm, vias 0 -> 52
- net /FPGA/FPGA.SCK: track 600.0 -> 116.9 mm, vias 0 -> 28
- net nRESET: track 510.0 -> 97.3 mm, vias 0 -> 30
- net /FPGA/Ctrl.audioSCL: track 500.0 -> 115.7 mm, vias 0 -> 40
- net /Rx Front End/rxQ2-: track 300.0 -> 62.6 mm, vias 0 -> 7
- net /FPGA/Tune.C6: track 200.0 -> 57.0 mm, vias 0 -> 14
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
Commit message: Phase 3C: Working maze search routing with target doors
Completed integration of room-based routing infrastructure:

* Target door generation:
  - Fixed search tree initialization (clear before populating)
  - Target doors properly created when rooms intersect items
  - Maze search successfully expands to target doors

* Room sizing optimization:
  - Reduced expansion from 1000mm to 2.5mm for better quality
  - Smaller rooms force multi-step pathfinding
  - Balanced routing success (525/1148 = 45.7%) with quality (7k DRC violations vs 17k)

* Infrastructure fixes:
  - Item now inherits from SearchTreeObject for spatial indexing
  - Search tree properly populated after initConnection() clears it
  - Room shapes preserved through completion process
  - Cleaned up verbose debug output

Results on NexRx test board:
- 525 items routed out of 1148 (45.7% success rate)
- 7,041 DRC violations (improved from 17,725)
- Routes are being found and traces inserted
- Quality issues remain (direct point-to-point, no obstacle avoidance yet)

Next steps:
- Implement proper obstacle avoidance in room shape completion
- Add intermediate waypoints for better path quality
- Enable room-to-room door generation for complex routes

🤖 Generated with [Claude Code](https://claude.com/claude-code)

Co-Authored-By: Claude <noreply@anthropic.com>
Routing:
- net +3.3V: track 2633.4 -> 314.4 mm, vias 719 -> 0
- net /FPGA/Ctrl.qsdSCK: track 163.6 -> 1894.5 mm, vias 59 -> 0
- net /FPGA/FPGA.NSS: track 162.9 -> 951.0 mm, vias 52 -> 0
- net /Rx Front End/Rx Preselector/preselIn: track 945.4 -> 233.5 mm, vias 208 -> 0
- net +3.3V-ON: track 627.9 -> 68.4 mm, vias 280 -> 0
- net /FPGA/Ctrl.audioSCL: track 115.7 -> 640.4 mm, vias 40 -> 0
- net /FPGA/FPGA.SCK: track 116.9 -> 631.7 mm, vias 28 -> 0
- net +3.3VFPGAIO: track 561.5 -> 59.3 mm, vias 193 -> 0
- net +2V5bias: track 833.4 -> 382.8 mm, vias 321 -> 0
- net /Rx Front End/rxQ2-: track 62.6 -> 413.8 mm, vias 7 -> 0
- net /FPGA/Tune.C4: track 52.0 -> 301.8 mm, vias 17 -> 0
- net /FPGA/VFPGAPLL: track 60.0 -> 276.8 mm, vias 24 -> 0
- net +VFPGACORE: track 209.3 -> 20.8 mm, vias 118 -> 0
- net /Rx Front End/rxI2+: track 34.9 -> 214.6 mm, vias 6 -> 0
- net /Power/usbDN: track 24.4 -> 171.6 mm, vias 8 -> 0
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